File: Main PCB/OutatimePro.kicad_pcb (KiCad board)
At the start: 2 copper layers, 25.7 x 27.7 mm, 43 parts, among them IC1 PAM8904JPR, J1 USB_B_Micro_PCB_Edge_receptac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, J2 FH35C-9S-0.3SHW, J3 TagConnect_TC2030-NL, Q1 ALS-PT19-315C/L177/TR8, SW1 EVPAWED40, U1 ATSAML22N18A-CFUT, U2 MIC5365-3.3YMT, U3 USBLC6-2P6, U4 MAX40200ANS, Y1 32.768kHz

Commit message: Add display clearance height
Other:
- board text added: "0.65mm"

Commit message: add display clearance text to footprint
Other:
- board text removed: "0.65mm"

Commit message: v270826: change programming header, add test points
Parts:
- added TP1: USB+, OutatimePro:TestPoint_Pad_D1.5mm, B.Cu at (33.2, 15.5)
- added TP2: USB-, OutatimePro:TestPoint_Pad_D1.5mm, B.Cu at (31.2, 15.0)
- added TP3: +3v3, OutatimePro:TestPoint_Pad_D1.5mm, B.Cu at (27.5, 21.5)
- added TP4: GND, OutatimePro:TestPoint_Pad_D1.5mm, B.Cu at (30.5, 30.0)
- J3: value TagConnect_TC2030-NL -> OSO_SWD; footprint Connector:Tag-Connect_TC2030-IDC-NL_2x03_P1.27mm_Vertical -> OutatimePro:OSO_SWD_2x3
- moved C10 1.10 mm to (17.5, 22.2)
- moved J3 0.71 mm to (22.2, 20.8), turned to -90 degrees
Connections:
- J3 pad 1: VCC -> /SWDIO
- J3 pad 2: /SWDIO -> GND
- J3 pad 3: /~{RESET} -> VCC
- J3 pad 5: GND -> /~{RESET}
Routing:
- net /SWDIO: track 17.0 -> 21.6 mm, vias 2 -> 3
- net Net-(J1-D+): track 4.94 -> 9.59 mm, vias 0 -> 1
- net Net-(J1-D-): track 5.11 -> 8.79 mm, vias 0 -> 1
- net /SWCLK: track 19.5 -> 21.8 mm, vias 2 -> 3
- net VCC: track 153.7 -> 151.5 mm
- net /~{RESET}: track 58.3 -> 60.4 mm, vias 2 -> 3
- net +3.3V: track 27.3 -> 29.2 mm
- net /LIGHTSENSE: track 30.8 -> 29.1 mm
- net GND: track 60.5 -> 59.3 mm, vias 30 -> 29
Other:
- board text added: "v270826"
- board text removed: "CLK"
- board text removed: "G"
- board text removed: "IO"
- board text removed: "RST"
- board text removed: "V"
- board text removed: "v250826"
