File: Main PCB/OutatimePro.kicad_sch (KiCad schematic)
At the start: 47 parts, among them IC1 PAM8904JPR, J1 USB_B_Micro_PCB_Edge_receptac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, J2 FH35C-9S-0.3SHW, J3 OSO_SWD, Q1 ALS-PT19-315C/L177/TR8, SW1 EVPAWED40, U1 ATSAML22N18A-CFUT, U2 MIC5365-3.3YMT, U3 USBLC6-2P6, U4 MAX40200ANS, Y1 32.768kHz

Commit message: rename kicad nets to row/columns t2b,l2r
Connections:
- net KPD_A1 renamed KPD_C4
- net KPD_A2 renamed KPD_C3
- net KPD_A3 renamed KPD_C2
- net KPD_A4 renamed KPD_C1
- net KPD_B1 renamed KPD_R1
- net KPD_B2 renamed KPD_R2
- net KPD_B3 renamed KPD_R3
- net KPD_B4 renamed KPD_R4
Changed lines of the file:
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@@
+		)
+	)
+	(label "KPD_C1"
+		(at 101.6 212.09 0)
+		(effects
+			(font
+				(size 1.27 1.27)
+			)
+			(justify left bottom)
 		)
 	)
@@
 		)
 	)
+	(label "KPD_C3"
+		(at 101.6 217.17 0)
+		(effects
+			(font
+				(size 1.27 1.27)
+			)
+			(justify left bottom)
+		)
+	)
 	(label "USB_N"
 		(at 104.14 190.5 0)
@@
 		)
 	)
-	(label "KPD_A3"
+	(label "KPD_C2"
 		(at 289.56 185.42 180)
 		(effects
@@
 		)
 	)
+	(label "KPD_R2"
+		(at 101.6 209.55 0)
+		(effects
+			(font
+				(size 1.27 1.27)
+			)
+			(justify left bottom)
+		)
+	)
 	(label "SEG18"
 		(at 243.84 166.37 180)
@@
 		)
 	)
+	(label "KPD_R1"
+		(at 101.6 198.12 0)
+		(effects
+			(font
+				(size 1.27 1.27)
+			)
+			(justify left bottom)
+		)
+	)
 	(label "BUZZER_DIN"
 		(at 342.9 227.33 180)
@@
 		)
 	)
-	(label "KPD_A1"
+	(label "KPD_C4"
 		(at 289.56 190.5 180)
 		(effects
@@
 		)
 	)
-	(label "KPD_A1"
-		(at 101.6 219.71 0)
-		(effects
-			(font
-				(size 1.27 1.27)
-			)
-			(justify left bottom)
-		)
-	)
-	(label "KPD_B4"
-		(at 101.6 207.01 0)
-		(effects
-			(font
-				(size 1.27 1.27)
-			)
-			(justify left bottom)
-		)
-	)
 	(label "~{BLUE}"
 		(at 373.38 139.7 180)
@@
 		)
 	)
+	(label "KPD_R4"
+		(at 101.6 207.01 0)
+		(effects
+			(font
+				(size 1.27 1.27)
+			)
+			(justify left bottom)
+		)
+	)
 	(label "SEG03"
 		(at 243.84 224.79 180)
@@
 		)
 	)
+	(label "KPD_R3"
+		(at 101.6 195.58 0)
+		(effects
+			(font
+				(size 1.27 1.27)
+			)
+			(justify left bottom)
+		)
+	)
 	(label "XIN32"
 		(at 104.14 163.83 0)
@@
 		)
 	)
+	(label "KPD_C4"
+		(at 101.6 219.71 0)
+		(effects
+			(font
+				(size 1.27 1.27)
+			)
+			(justify left bottom)
+		)
+	)
 	(label "SEG07"
 		(at 243.84 212.09 180)
@@
 		)
 	)
-	(label "KPD_B3"
-		(at 101.6 195.58 0)
-		(effects
-			(font
-				(size 1.27 1.27)
-			)
-			(justify left bottom)
-		)
-	)
-	(label "KPD_A2"
-		(at 101.6 217.17 0)
+	(label "KPD_C2"
+		(at 101.6 214.63 0)
 		(effects
 			(font
@@
 		)
 	)
-	(label "KPD_B1"
+	(label "KPD_R1"
 		(at 289.56 180.34 180)
 		(effects
@@
 		)
 	)
-	(label "KPD_B3"
+	(label "KPD_R3"
 		(at 289.56 175.26 180)
 		(effects
@@
 			)
 			(justify right bottom)
-		)
-	)
-	(label "KPD_B1"
-		(at 101.6 198.12 0)
-		(effects
-			(font
-				(size 1.27 1.27)
-			)
-			(justify left bottom)
 		)
 	)
@@
 		)
 	)
-	(label "KPD_B2"
+	(label "KPD_R2"
 		(at 289.56 177.8 180)
 		(effects
@@
 		)
 	)
-	(label "KPD_A4"
-		(at 101.6 212.09 0)
-		(effects
-			(font
-				(size 1.27 1.27)
-			)
-			(justify left bottom)
-		)
-	)
 	(label "SEG10"
 		(at 289.56 97.79 180)
@@
 		)
 	)
-	(label "KPD_A3"
-		(at 101.6 214.63 0)
-		(effects
-			(font
-				(size 1.27 1.27)
-			)
-			(justify left bottom)
-		)
-	)
-	(label "KPD_A2"
+	(label "KPD_C3"
 		(at 289.56 187.96 180)
 		(effects
@@
 		)
 	)
-	(label "KPD_A4"
+	(label "KPD_C1"
 		(at 289.56 182.88 180)
 		(effects
@@
 		)
 	)
-	(label "KPD_B4"
+	(label "KPD_R4"
 		(at 289.56 172.72 180)
 		(effects
@@
 		)
 	)
-	(label "KPD_B2"
-		(at 101.6 209.55 0)
-		(effects
-			(font
-				(size 1.27 1.27)
-			)
-			(justify left bottom)
-		)
-	)
