File: Accelerometer FPC/OutatimeProAccelerometer.kicad_sch (KiCad schematic)
At the start: 4 parts, among them J1 FH35C-9S-0.3SHW, U1 LIS2DW12TR

Commit message: remove lcd mapping pcb and add lcsc component numbers to fpc board
Parts:
- C1: LCSC Part # (none) -> C19702
- C2: LCSC Part # (none) -> C14663
- J1: LCSC Part # C189624 -> (none)
- U1: LCSC Part # (none) -> C189624
Changed lines of the file:
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@@
 		(in_bom no)
 		(on_board yes)
-		(in_pos_files yes)
+		(in_pos_files no)
 		(dnp no)
 		(fields_autoplaced yes)
@@
 			)
 		)
-		(property "LCSC Part #" "C189624"
+		(property "LCSC Part #" ""
 			(at 58.42 46.99 0)
 			(hide yes)
@@
 			)
 		)
+		(property "LCSC Part #" "C189624"
+			(at 44.45 91.44 0)
+			(hide yes)
+			(show_name no)
+			(do_not_autoplace no)
+			(effects
+				(font
+					(size 1.27 1.27)
+				)
+			)
+		)
 		(pin "10"
 		)
@@
 			)
 		)
-		(property "LCSC Part #" ""
+		(property "LCSC Part #" "C19702"
 			(at 82.55 80.01 0)
 			(hide yes)
@@
 			)
 		)
-		(property "LCSC Part #" ""
+		(property "LCSC Part #" "C14663"
 			(at 71.12 80.01 0)
 			(hide yes)
